File: sa612/sa612.sch (KiCad schematic (older format))
At the start: 11 parts, among them J1 RF_IN, J2 PWR, J3 OSC_IN, J4 IF_OUT, U1 SA612, U2 MCP1700-5002E_SOT23

Commit message: Clean up commit
Parts:
- added C6: 10uF, Capacitors_SMD:C_1206_HandSoldering, symbol Device:CP
- C3: value 10uF -> 1uF
- U2: footprint Package_TO_SOT_SMD:SOT-23 -> TO_SOT_Packages_SMD:SOT-23
Connections:
- wire segments 39 -> 43
Changed lines of the file:
@@
 P 1900 1400
 F 0 "C3" V 1645 1400 50  0000 C CNN
-F 1 "10uF" V 1736 1400 50  0000 C CNN
+F 1 "1uF" V 1736 1400 50  0000 C CNN
 F 2 "Capacitors_SMD:C_1206_HandSoldering" H 1938 1250 50  0001 C CNN
 F 3 "~" H 1900 1400 50  0001 C CNN
@@
 F 0 "U2" H 2950 1492 50  0000 C CNN
 F 1 "MCP1700-5002E_SOT23" H 2950 1401 50  0000 C CNN
-F 2 "Package_TO_SOT_SMD:SOT-23" H 2950 1475 50  0001 C CNN
+F 2 "TO_SOT_Packages_SMD:SOT-23" H 2950 1475 50  0001 C CNN
 F 3 "http://ww1.microchip.com/downloads/en/DeviceDoc/20001826C.pdf" H 2950 1250 50  0001 C CNN
 	1    2950 1250
@@
 $EndComp
 Wire Wire Line
-	3650 1250 3250 1250
+	3650 1250 3350 1250
 Wire Wire Line
 	3650 1350 3500 1350
+Connection ~ 3500 1650
+Wire Wire Line
+	2950 1650 3350 1650
+Wire Wire Line
+	2950 1550 2950 1650
+$Comp
+L Device:CP C6
+U 1 1 5B6C4B57
+P 3350 1450
+F 0 "C6" H 3468 1496 50  0000 L CNN
+F 1 "10uF" H 3468 1405 50  0000 L CNN
+F 2 "Capacitors_SMD:C_1206_HandSoldering" H 3388 1300 50  0001 C CNN
+F 3 "~" H 3350 1450 50  0001 C CNN
+	1    3350 1450
+	1    0    0    -1
+$EndComp
 Wire Wire Line
 	3500 1350 3500 1650
-Connection ~ 3500 1650
-Wire Wire Line
-	2950 1650 3500 1650
-Wire Wire Line
-	2950 1550 2950 1650
+Wire Wire Line
+	3350 1300 3350 1250
+Connection ~ 3350 1250
+Wire Wire Line
+	3350 1250 3250 1250
+Wire Wire Line
+	3350 1600 3350 1650
+Connection ~ 3350 1650
+Wire Wire Line
+	3350 1650 3500 1650
 $EndSCHEMATC

Commit message: Fix the sa612 board layout
Parts:
- removed U2: MCP1700-5002E_SOT23, TO_SOT_Packages_SMD:SOT-23, symbol Regulator_Linear:MCP1700-5002E_SOT23
- added U2: LD1117S50TR_SOT223, TO_SOT_Packages_SMD:SOT-223-3_TabPin2, symbol Regulator_Linear:LD1117S50TR_SOT223
- OUT1: renamed from J4; value IF_OUT -> RF_OUT
- renumbered J3 to IF1, J1 to IN1
Changed lines of the file:
@@
 EESchema Schematic File Version 4
+LIBS:sa612-cache
 EELAYER 26 0
 EELAYER END
@@
 	3500 2950 2350 2950
 $Comp
-L Connector_Generic:Conn_01x03 J3
+L Connector_Generic:Conn_01x03 IF1
 U 1 1 5B6B9B1D
 P 3850 1750
-F 0 "J3" H 3929 1792 50  0000 L CNN
+F 0 "IF1" H 3929 1792 50  0000 L CNN
 F 1 "OSC_IN" H 3929 1701 50  0000 L CNN
 F 2 "x-uhf:X-UHF_Interconnect" H 3850 1750 50  0001 C CNN
@@
 $EndComp
 $Comp
-L Connector_Generic:Conn_01x03 J4
+L Connector_Generic:Conn_01x03 OUT1
 U 1 1 5B6B9B76
 P 3850 2400
-F 0 "J4" H 3929 2442 50  0000 L CNN
-F 1 "IF_OUT" H 3929 2351 50  0000 L CNN
+F 0 "OUT1" H 3929 2442 50  0000 L CNN
+F 1 "RF_OUT" H 3929 2351 50  0000 L CNN
 F 2 "x-uhf:X-UHF_Interconnect" H 3850 2400 50  0001 C CNN
 F 3 "~" H 3850 2400 50  0001 C CNN
@@
 Connection ~ 3500 2500
 $Comp
-L Connector_Generic:Conn_01x03 J1
+L Connector_Generic:Conn_01x03 IN1
 U 1 1 5B6B9D7C
 P 700 2200
-F 0 "J1" H 620 1875 50  0000 C CNN
+F 0 "IN1" H 620 1875 50  0000 C CNN
 F 1 "RF_IN" H 620 1966 50  0000 C CNN
 F 2 "x-uhf:X-UHF_Interconnect" H 700 2200 50  0001 C CNN
@@
 	2350 1250 2350 1400
 Connection ~ 2350 1400
-$Comp
-L Regulator_Linear:MCP1700-5002E_SOT23 U2
-U 1 1 5B6BE2D2
-P 2950 1250
-F 0 "U2" H 2950 1492 50  0000 C CNN
-F 1 "MCP1700-5002E_SOT23" H 2950 1401 50  0000 C CNN
-F 2 "TO_SOT_Packages_SMD:SOT-23" H 2950 1475 50  0001 C CNN
-F 3 "http://ww1.microchip.com/downloads/en/DeviceDoc/20001826C.pdf" H 2950 1250 50  0001 C CNN
-	1    2950 1250
-	-1   0    0    -1
-$EndComp
 Wire Wire Line
 	2350 1250 2650 1250
@@
 Wire Wire Line
 	3350 1650 3500 1650
+$Comp
+L Regulator_Linear:LD1117S50TR_SOT223 U2
+U 1 1 5B721F22
+P 2950 1250
+F 0 "U2" H 2950 1492 50  0000 C CNN
+F 1 "LD1117S50TR_SOT223" H 2950 1401 50  0000 C CNN
+F 2 "TO_SOT_Packages_SMD:SOT-223-3_TabPin2" H 2950 1450 50  0001 C CNN
+F 3 "http://www.st.com/st-web-ui/static/active/en/resource/technical/document/datasheet/CD00000544.pdf" H 3050 1000 50  0001 C CNN
+	1    2950 1250
+	-1   0    0    -1
+$EndComp
 $EndSCHEMATC
