File: bfr93-amplifier/bfr93-amplifier.sch (KiCad schematic (older format))
At the start: 11 parts, among them J1 IN, J2 PWR, J3 OUT, Q1 BFR93A

Commit message: Add power decoupling for amplifier
Parts:
- added C?: 10u, Capacitors_SMD:C_1206_HandSoldering, symbol Device:C
Connections:
- wire segments 37 -> 40
Changed lines of the file:
@@
 EESchema Schematic File Version 4
+LIBS:bfr93-amplifier-cache
 EELAYER 26 0
 EELAYER END
@@
 	3250 1250 3650 1250
 Wire Wire Line
-	3650 1250 3650 1850
+	3650 1250 3650 1450
 Connection ~ 3650 1850
+$Comp
+L Device:C C?
+U 1 1 5B82EA62
+P 3200 1450
+F 0 "C?" V 2948 1450 50  0000 C CNN
+F 1 "10u" V 3039 1450 50  0000 C CNN
+F 2 "Capacitors_SMD:C_1206_HandSoldering" H 3238 1300 50  0001 C CNN
+F 3 "~" H 3200 1450 50  0001 C CNN
+	1    3200 1450
+	0    1    1    0
+$EndComp
+Wire Wire Line
+	3050 1450 2800 1450
+Wire Wire Line
+	3350 1450 3650 1450
+Connection ~ 3650 1450
+Wire Wire Line
+	3650 1450 3650 1850
 $EndSCHEMATC

Commit message: FM demodulator and interface
Parts:
- gave numbers to parts that had none: 1
Changed lines of the file:
@@
 Connection ~ 3650 1850
 $Comp
-L Device:C C?
+L Device:C C4
 U 1 1 5B82EA62
 P 3200 1450
-F 0 "C?" V 2948 1450 50  0000 C CNN
+F 0 "C4" V 2948 1450 50  0000 C CNN
 F 1 "10u" V 3039 1450 50  0000 C CNN
 F 2 "Capacitors_SMD:C_1206_HandSoldering" H 3238 1300 50  0001 C CNN
